File: files/kicad/SLiCAP.kicad_sch (KiCad schematic)
At the start: 36 parts

Commit message: Added missing CSS file
Parts:
- added O1: ~, symbol SLiCAP:O
- A? (x2), D?, J?, M?, N?, Q?, X? (x14): value (none) -> ~

Commit message: Improved windows installation
Parts:
- removed X?: ~, symbol SLiCAP:O_noise
- added X1: ~, symbol SLiCAP:O_noise
- added X2: ~, symbol SLiCAP:Xio5
- added X3: ~, symbol SLiCAP:Xamp3
- added X5: ~, symbol SLiCAP:Xamp4
- added X6: ~, symbol SLiCAP:Xamp5
- added X7: ~, symbol SLiCAP:Xio3
- added X8: ~, symbol SLiCAP:Xio4
